Commit message: drop visual/geometry elements in test URDFs, silence test-time warnings
And while at it, might as well drop the 'inertial' and 'ros2_control'
elements to save some lines

File: crx_kinematics/test/crx10ia.urdf (robot description, URDF)
Before this commit: robot crx10ia, 11 links, 10 joints
Links:
- link J1_link: mass 10.673 -> None; geometry 
- link J2_link: mass 10.892 -> None; geometry 
- link J3_link: mass 4.162 -> None; geometry 
- link J4_link: mass 3.969 -> None; geometry 
- link J5_link: mass 2.509 -> None; geometry 
- link J6_link: mass 1.305 -> None; geometry 
- link base_link: mass 4.517 -> None; geometry 

File: crx_kinematics/test/crx30ia.urdf (robot description, URDF)
Before this commit: robot crx30ia, 11 links, 10 joints
Links:
- link J1_link: mass 41.083 -> None; geometry 
- link J2_link: mass 41.783 -> None; geometry 
- link J3_link: mass 11.493 -> None; geometry 
- link J4_link: mass 10.453 -> None; geometry 
- link J5_link: mass 4.247 -> None; geometry 
- link J6_link: mass 2.075 -> None; geometry 
- link base_link: mass 21.685 -> None; geometry 
